Commit message: Add Foxy RViz arm joint control

File: upper_computer_ws/src/humanoid_arm_description/urdf/humanoid_arm.urdf (robot description, URDF)
Before this commit: robot humanoid_arm, 7 links, 6 joints
Links:
- link link_1: geometry collision cylinder length=0.05775 radius=0.006; visual cylinder length=0.05775 radius=0.006
- link link_2: geometry collision cylinder length=0.07 radius=0.006; visual cylinder length=0.07 radius=0.006
- link link_3: geometry collision cylinder length=0.035 radius=0.0055; visual cylinder length=0.035 radius=0.0055
- link link_4: geometry collision sphere radius=0.009; visual sphere radius=0.009

Commit message: Fix arm zero-pose joint geometry

File: upper_computer_ws/src/humanoid_arm_description/urdf/humanoid_arm.urdf (robot description, URDF)
Before this commit: robot humanoid_arm, 7 links, 6 joints
Links:
- link link_1: geometry collision cylinder length=0.05 radius=0.006; visual cylinder length=0.05 radius=0.006
- link tool_link: geometry collision sphere radius=0.006; visual sphere radius=0.006
Joints:
- joint joint_1: axis 0 0 1 -> 0 0.5 0.8660254; origin xyz=0.002 0.003 0 rpy=-1.57079632679 0 0 -> xyz=0 0 0 rpy=0 0 0
- joint joint_2: axis 0 0 1 -> 1 0 0; origin xyz=0.0289 -0.05 0 rpy=1.57079632679 0 0 -> xyz=0 -0.05 0 rpy=0 0 0
- joint joint_3: origin xyz=0 0.07 0 rpy=-1.57079632679 0 0 -> xyz=0 0 -0.07 rpy=0 0 0
- joint joint_4: axis 0 0 1 -> 0 1 0; origin xyz=0 -0.035 0 rpy=1.57079632679 0 0 -> xyz=0 0 -0.035 rpy=0 0 0

Commit message: refactor: 调整基座轴线与关节位置, 添加末端杆及6-DOF显示
- 基座轴线改为Rx(60°)指向(0,-√3/2,1/2)，joint_2零点保持竖直
- 基座顶面/joint_1移至(0,0,0)，link_1=50mm时joint_2在(0,-50mm,0)
- 关节颜色改为红色(joint_red)与连杆区分
- 添加270mm末端杆(end_rod)+tip_frame
- 新增tip_position_gui.py：tkinter窗口实时显示末端位置+姿态(RPY)

File: upper_computer_ws/src/humanoid_arm_description/urdf/humanoid_arm.urdf (robot description, URDF)
Before this commit: robot humanoid_arm, 7 links, 6 joints
Links:
- added link end_rod, mass 0.08; collision cylinder length=0.27 radius=0.005; visual cylinder length=0.27 radius=0.005
- added link tip_frame
- link link_1: geometry collision cylinder length=0.05 radius=0.006; visual cylinder length=0.02 radius=0.008
- link link_2: geometry collision cylinder length=0.07 radius=0.006; visual cylinder length=0.02 radius=0.008
- link link_3: geometry collision cylinder length=0.035 radius=0.0055; visual cylinder length=0.018 radius=0.007
- link link_4: geometry collision sphere radius=0.009; visual cylinder length=0.018 radius=0.007
Joints:
- added joint rod_joint: type fixed, parent link_4, child end_rod
- added joint tip_joint: type fixed, parent end_rod, child tip_frame, origin xyz=0 0 -0.27 rpy=0 0 0
- joint joint_1: axis 0 0.5 0.8660254 -> 0 0 1; limit lower=-1.483529864 upper=3.054326191 effort=10 velocity=3.141592654 -> lower=-3.141592654 upper=3.141592654 effort=10 velocity=3.141592654
- joint joint_2: limit lower=-0.174532925 upper=2.617993878 effort=10 velocity=3.141592654 -> lower=-3.141592654 upper=3.141592654 effort=10 velocity=3.141592654; origin xyz=0 -0.05 0 rpy=0 0 0 -> xyz=0 -0.05 0 rpy=-1.047197551 0 0
- joint joint_3: limit lower=-1.745329252 upper=1.745329252 effort=10 velocity=3.141592654 -> lower=-3.141592654 upper=3.141592654 effort=10 velocity=3.141592654
- joint joint_4: limit lower=-0.698131701 upper=1.745329252 effort=10 velocity=3.141592654 -> lower=-3.141592654 upper=3.141592654 effort=10 velocity=3.141592654
- joint world_joint: origin (none) -> xyz=0 0 0 rpy=1.047197551 0 0

Commit message: fix: align arm URDF with joint geometry

File: upper_computer_ws/src/humanoid_arm_description/urdf/humanoid_arm.urdf (robot description, URDF)
Before this commit: robot humanoid_arm, 9 links, 8 joints
Joints:
- joint joint_1: axis 0 0 1 -> 0 -0.8660254 0.5
- joint joint_2: origin xyz=0 -0.05 0 rpy=-1.047197551 0 0 -> xyz=0 -0.05 0 rpy=0 0 0
- joint world_joint: origin xyz=0 0 0 rpy=1.047197551 0 0 -> xyz=0 0 0 rpy=0 0 0
